Commit message: Added RTAB-map functionality
Modified robot .gazebo file to include an rgbd camera. Created a
mapping.launch file for the ROS rtabmap node and parameters.

File: catkin_ws/src/my_robot/urdf/my_robot.xacro (robot description, xacro)
@@ -232,4 +232,6 @@
     </visual>
   </link>
+  <link name="camera_link_optical">
+  </link>
   <link name="hokuyo">
     <origin xyz="0 0 0" rpy="0 0 0"/>
@@ -289,4 +291,9 @@
     <axis xyz="0 1 0" rpy="0 0 0"/>
   </joint>
+  <joint type="fixed" name="camera_optical_joint">
+    <origin xyz="0 0 0" rpy="-1.5707 0 -1.5707"/>
+    <child link="camera_link_optical"/>
+    <parent link="camera"/>
+  </joint>
   <joint type="fixed" name="hokuyo_joint">
     <origin xyz="0.2 0 0.12" rpy="0 0 0"/>
